File: DIY-Arduino-PCB/DIY-Arduino-PCB.kicad_sch (KiCad schematic)
At the start: 5 parts, among them J2 USB_C_Receptacle_USB2.0_16P, U1 RP2350A, U2 ATmega328P-M, U3 ESP32-C3, U4 USBLC6-2SC6

Commit message: Added some basic USB Circuitry
Parts:
- removed U2: ATmega328P-M, Package_DFN_QFN:QFN-32-1EP_5x5mm_P0.5mm_EP3.1x3.1mm, symbol MCU_Microchip_ATmega:ATmega328P-M
- removed U3: ESP32-C3, Package_DFN_QFN:QFN-32-1EP_5x5mm_P0.5mm_EP3.7x3.7mm, symbol MCU_Espressif:ESP32-C3
- added C1, C2: 20pf, symbol Device:C
- added C3, C4, C5, C6, C7, C8, C9: C, symbol Device:C
- added F1: Polyfuse, symbol Device:Polyfuse
- added FB1: FerriteBead, symbol Device:FerriteBead
- added J1: USB_C_Receptacle_USB2.0_16P, symbol Connector:USB_C_Receptacle_USB2.0_16P
- added R1, R2, R3, R4: R, symbol Device:R
- added SW1: SW_Push, symbol Switch:SW_Push
- added U2: ATmega16U2-A, Package_QFP:TQFP-32_7x7mm_P0.8mm, symbol MCU_Microchip_ATmega:ATmega16U2-A
- added U3: ESP32-S3, Package_DFN_QFN:QFN-56-1EP_7x7mm_P0.4mm_EP4x4mm, symbol MCU_Espressif:ESP32-S3
- added U5: ATmega328P-M, Package_DFN_QFN:QFN-32-1EP_5x5mm_P0.5mm_EP3.1x3.1mm, symbol MCU_Microchip_ATmega:ATmega328P-M
- added U6: CH340G, Package_SO:SOIC-16_3.9x9.9mm_P1.27mm, symbol Interface_USB:CH340G
- added Y1: 16MHz, symbol Device:Crystal
- added Y2, Y3: Crystal, symbol Device:Crystal
Connections:
- net GND: now also C1.2, C2.1, C3.1, C4.2, C5.2, C6.1, C8.2, C9.2, SW1.2, U2.3 (GND), U3.57 (GND), U5.21 (GND), U5.3 (GND), U5.33 (GND), U5.5 (GND)
- new net: C5.1, U5.8 (XTAL2/PB7), Y2.1
- new net: C1.1, R1.2, U2.2 (PC0/XTAL2), Y1.2
- new net: J1.A1 (GND), J1.A12 (GND), J1.B1 (GND), J1.B12 (GND)
- new net: F1.1, J1.A4 (VBUS), J1.A9 (VBUS), J1.B4 (VBUS), J1.B9 (VBUS)
- new net: J1.A6 (D+), J1.B6 (D+), R3.1
- new net: J1.A7 (D-), J1.B7 (D-), R4.1
- new net: C4.1, U5.7 (XTAL1/PB6), Y2.2
- new net: C8.1, U6.8 (XO), Y3.2
- new net: C2.2, R1.1, U2.1 (XTAL1), Y1.1
- new net: C7.1, F1.2, FB1.1
- new net: R4.2, U6.6 (UD-)
- new net: R3.2, U6.5 (UD+)
- new net: C9.1, U6.7 (XI), Y3.1
- new net: U3.2 (VDD3P3), U3.3 (VDD3P3)
- new net: U3.55 (VDDA), U3.56 (VDDA)
- new net: R2.1, SW1.1, U5.29 (~{RESET}/PC6)
- new net +5V: C3.2, C6.2, C7.2, FB1.2, R2.2, U2.32 (AVCC), U2.4 (VCC), U5.18 (AVCC), U5.4 (VCC), U5.6 (VCC)
- new net RX: U5.30 (PD0), U6.3 (RXD)
- new net TX: U5.31 (PD1), U6.2 (TXD)
Other:
- note added: "ATMEL: 1. Clock - 16 MHz with 2 caps- 1 on each terminal connected to GND connect Clock to XTAL 1/2 pins. 1 megaohm resistor in parallel with the crystal 2. Power - Decoupling cap of 100nF at VCC and AVCC 3."
- moved on the sheet: J2, U1, U4

Commit message: did USB stuff
Parts:
- removed C1, C2: 20pf, symbol Device:C
- removed C3: C, symbol Device:C
- removed J2: USB_C_Receptacle_USB2.0_16P, symbol Connector:USB_C_Receptacle_USB2.0_16P
- removed R1: R, symbol Device:R
- removed U1: RP2350A, Package_DFN_QFN:QFN-60-1EP_7x7mm_P0.4mm_EP3.4x3.4mm, symbol MCU_RaspberryPi:RP2350A
- removed U2: ATmega16U2-A, Package_QFP:TQFP-32_7x7mm_P0.8mm, symbol MCU_Microchip_ATmega:ATmega16U2-A
- removed U3: ESP32-S3, Package_DFN_QFN:QFN-56-1EP_7x7mm_P0.4mm_EP4x4mm, symbol MCU_Espressif:ESP32-S3
- removed U4: USBLC6-2SC6, Package_TO_SOT_SMD:SOT-23-6, symbol Power_Protection:USBLC6-2SC6
- removed Y1: 16MHz, symbol Device:Crystal
- added C10, C11, C12: 0.1uf, symbol Device:C
- added D1, D2, D3, D4: LED, symbol Device:LED
- added R5: 1M, symbol Device:R
- added R6, R7, R8, R9: R, symbol Device:R
- C7: value C -> 10uf
- R3, R4: value R -> 22
Connections:
- net +5V: now also C7.1, U6.16 (VCC), C10.2, R6.1; no longer C7.2
- net GND: now also C7.2, J1.A1 (GND), J1.A12 (GND), J1.B1 (GND), J1.B12 (GND), U6.1 (GND), C10.1, C12.2, D1.1 (K), D2.1 (K), D3.1 (K), D4.1 (K), R5.2
- net RX: now also U6.2 (TXD); no longer U6.3 (RXD)
- net TX: now also U6.3 (RXD); no longer U6.2 (TXD)
- net at J1.S1 (SHIELD): now also R5.1
- net at F1.2, FB1.1: no longer C7.1
- net at U6.13 (~{DTR}): now also C11.1
- net at U6.4 (V3): now also C12.1
- net RST: now reaches R2.1, SW1.1, U5.29 (~{RESET}/PC6)
- net RST: now also C11.2
- new net: D3.2 (A), R8.2
- new net: D4.2 (A), R9.2
- new net: D2.2 (A), R7.2
- new net: D1.2 (A), R6.2
Other:
- note added: "Power Status Tx/Rx LEDs Blinky"
- note added: "Status LEDs"
- note added: "TX and RX are swapped here bc we need to communicate if they weren't, the usb would send data on Tx and the arduino woudl also try to send data on Tx and anything they sent to each other would get caught going nowhere"
- note removed: "ATMEL"
- note removed: "ATMEL: 1. Clock - 16 MHz with 2 caps- 1 on each terminal connected to GND connect Clock to XTAL 1/2 pins. 1 megaohm resistor in parallel with the crystal 2. Power - Decoupling cap of 100nF at VCC and AVCC 3."
- note removed: "ESP32"
- note removed: "RP2350"
- moved on the sheet: C7

Commit message: made some progress. Some odds and ends.
Parts:
- removed D2, D3: LED, symbol Device:LED
- removed R7, R8: R, symbol Device:R
- added H1, H2, H3, H4: MountingHole, symbol Mechanical:MountingHole
- added J2, J5: Conn_02x08_Top_Bottom, Connector_JAE:JAE_LY20-16P-DLT1_2x08_P2.00mm_Horizontal, symbol Connector_Generic:Conn_02x08_Top_Bottom
- added J3: Conn_02x06_Top_Bottom, symbol Connector_Generic:Conn_02x06_Top_Bottom
- added J4: Conn_02x03_Top_Bottom, symbol Connector_Generic:Conn_02x03_Top_Bottom
- C6: value C -> 0.1uF
Connections:
- net +5V: now also J4.1 (Pin_1)
- net GND: now also J2.10 (Pin_10), J2.11 (Pin_11), J2.12 (Pin_12), J2.13 (Pin_13), J2.14 (Pin_14), J2.15 (Pin_15), J2.16 (Pin_16), J2.9 (Pin_9), J3.10 (Pin_10), J3.11 (Pin_11), J3.12 (Pin_12), J3.7 (Pin_7), J3.8 (Pin_8), J3.9 (Pin_9), J4.3 (Pin_3), J5.10 (Pin_10), J5.11 (Pin_11), J5.12 (Pin_12), J5.13 (Pin_13), J5.14 (Pin_14), J5.15 (Pin_15), J5.16 (Pin_16), J5.9 (Pin_9)
- net RST: now also J4.6 (Pin_6)
- net RX: now also J2.1 (Pin_1)
- net TX: now also J2.2 (Pin_2)
- net D13: now reaches R9.1
- net D13: now also U5.17 (PB5), J3.6 (Pin_6), J4.5 (Pin_5)
- net D3: now reaches U5.1 (PD3)
- net D3: now also J2.4 (Pin_4)
- net D6: now reaches U5.10 (PD6)
- net D6: now also J2.7 (Pin_7)
- net D7: now reaches U5.11 (PD7)
- net D7: now also J2.8 (Pin_8)
- net D8: now reaches U5.12 (PB0)
- net D8: now also J3.1 (Pin_1)
- net D9(PWM): now reaches U5.13 (PB1)
- net D9(PWM): now also J3.2 (Pin_2)
- net D10(PWM): now reaches U5.14 (PB2)
- net D10(PWM): now also J3.3 (Pin_3)
- net D11(PWM): now reaches U5.15 (PB3)
- net D11(PWM): now also J3.4 (Pin_4)
- net D12: now reaches U5.16 (PB4)
- net D12: now also J3.5 (Pin_5), J4.4 (Pin_4)
- net A6: now reaches U5.19 (ADC6)
- net A6: now also J5.7 (Pin_7)
- net D4: now reaches U5.2 (PD4)
- net D4: now also J2.5 (Pin_5)
- net AREF: now reaches U5.20 (AREF)
- net A7: now reaches U5.22 (ADC7)
- net A7: now also J5.8 (Pin_8)
- net A0: now reaches U5.23 (PC0)
- net A0: now also J5.1 (Pin_1)
- net A1: now reaches U5.24 (PC1)
- net A1: now also J5.2 (Pin_2)
- net A2: now reaches U5.25 (PC2)
- net A2: now also J5.3 (Pin_3)
- net A3: now reaches U5.26 (PC3)
- net A3: now also J5.4 (Pin_4)
- net A4/SDA: now reaches U5.27 (PC4)
- net A4/SDA: now also J5.5 (Pin_5)
- net A5/SCL: now reaches U5.28 (PC5)
- net A5/SCL: now also J5.6 (Pin_6)
- net D2: now reaches U5.32 (PD2)
- net D2: now also J2.3 (Pin_3)
- net D5: now reaches U5.9 (PD5)
- net D5: now also J2.6 (Pin_6)
- new net D11: J4.2 (Pin_2)
Other:
- note added: "Blinky"
- note added: "Connectors"
- note added: "ICSP Connector"
- note added: "MCU"
- note added: "Mechanical"
- note added: "Power status"
- note added: "USB"
- note removed: "Power Status Tx/Rx LEDs Blinky"
- moved on the sheet: C10, C11, C12, C4, C5, C6, C7, C8, C9, D1, F1, FB1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
